File: hardware/DIY3/firebeetle-shield-v1/firebeetle-shield.kicad_sch (KiCad schematic)
At the start: 8 parts, among them J1 Conn_01x14_Female, J2 Conn_01x06_Female (DS3231), J3 Conn_01x04_Male (MS5803), J4 Conn_01x06_Female (microSD), J5 Conn_01x18_Female

Commit message: Add revision info
Other:
- title: (none) -> DIY3 FireBeetle Shield
Changed lines of the file:
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@@
 (kicad_sch (version 20211123) (generator eeschema)
   (paper "A4")
+  (title_block
+    (title "DIY3 FireBeetle Shield")
+    (date "2022-06-08")
+    (rev "v1")
+  )
   (wire (pts (xy 104.14 53.34) (xy 115.57 53.34))
     (stroke (width 0) (type default) (color 0 0 0 0))
