File: hardware/DIY4/firebeetle-shield/firebeetle-shield.kicad_sch (KiCad schematic)
At the start: 11 parts, among them J1 Conn_01x14_Female, J2 Conn_01x18_Female, J3 Conn_01x06_Female, J4 Conn_01x04_Male, J5 Conn_01x06_Female, Q1 Q_PJFET_GSD

Commit message: Commit some changes that have been sitting around for a while
Changed lines of the file:
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@@
 (kicad_sch
-	(version 20231120)
+	(version 20250114)
 	(generator "eeschema")
-	(generator_version "8.0")
+	(generator_version "9.0")
 	(paper "A4")
 	(title_block
@@
 		(rev "v2")
 	)
+	(text "MS5803 Pin Header"
+		(exclude_from_sim no)
+		(at 77.47 15.24 0)
+		(effects
+			(font
+				(size 1.27 1.27)
+			)
+			(justify left bottom)
+		)
+	)
+	(text "I2C Pull-Up Resistors"
+		(exclude_from_sim no)
+		(at 137.16 15.24 0)
+		(effects
+			(font
+				(size 1.27 1.27)
+			)
+			(justify left bottom)
+		)
+	)
+	(text "DS3231 Pin Header"
+		(exclude_from_sim no)
+		(at 77.47 38.1 0)
+		(effects
+			(font
+				(size 1.27 1.27)
+			)
+			(justify left bottom)
+		)
+	)
+	(text "Micro SD Pin Header\n(with optional high side MOSFET switch which can be \nenabled/disabled using the solder bridge)"
+		(exclude_from_sim no)
+		(at 77.47 82.55 0)
+		(effects
+			(font
+				(size 1.27 1.27)
+			)
+			(justify left bottom)
+		)
+	)
+	(text "Shield Pin Headers\nNote: SDA1 and SDA2 (and SCL1 and SCL2) are actually \nconnected to each other on the FireBeetle 2 (i.e. they are \nthe same I2C channels, just exposed on the pin headers in \ntwo different places)."
+		(exclude_from_sim no)
+		(at 12.7 22.86 0)
+		(effects
+			(font
+				(size 1.27 1.27)
+			)
+			(justify left bottom)
+		)
+	)
 	(junction
 		(at 102.87 111.76)
@@
 			(width 0)
 			(type dash)
-		)
-	)
-	(text "MS5803 Pin Header"
-		(exclude_from_sim no)
-		(at 77.47 15.24 0)
-		(effects
-			(font
-				(size 1.27 1.27)
-			)
-			(justify left bottom)
-		)
-	)
-	(text "I2C Pull-Up Resistors"
-		(exclude_from_sim no)
-		(at 137.16 15.24 0)
-		(effects
-			(font
-				(size 1.27 1.27)
-			)
-			(justify left bottom)
-		)
-	)
-	(text "DS3231 Pin Header"
-		(exclude_from_sim no)
-		(at 77.47 38.1 0)
-		(effects
-			(font
-				(size 1.27 1.27)
-			)
-			(justify left bottom)
-		)
-	)
-	(text "Micro SD Pin Header\n(with optional high side MOSFET switch which can be \nenabled/disabled using the solder bridge)"
-		(exclude_from_sim no)
-		(at 77.47 82.55 0)
-		(effects
-			(font
-				(size 1.27 1.27)
-			)
-			(justify left bottom)
-		)
-	)
-	(text "Shield Pin Headers\nNote: SDA1 and SDA2 (and SCL1 and SCL2) are actually \nconnected to each other on the FireBeetle 2 (i.e. they are \nthe same I2C channels, just exposed on the pin headers in \ntwo different places)."
-		(exclude_from_sim no)
-		(at 12.7 22.86 0)
-		(effects
-			(font
-				(size 1.27 1.27)
-			)
-			(justify left bottom)
 		)
 	)
@@
 		)
 	)
+	(embedded_fonts no)
 )
